File: TrebleSynth/TrebleSynth.kicad_pcb (KiCad board)
At the start: 2 copper layers, 236 x 128 mm, 220 parts, among them J1 INPUT, J10 DIN-5_180degree, J11 DIN-5_180degree, J2 INPUT, J3 OUTPUT, J5 Barrel_Jack_Switch, J8 INPUT, J9 INPUT, Q1 2N3904, Q2 2N3904, Q3 2N3904, Q4 2N3904, Q5 2N3904, Q6 2N3904, SW1 SW_Push, SW10 SW_Push, SW11 SW_Push, SW12 SW_Push, SW13 SW_Push, SW14 SW_Push, SW15 SW_Push, SW16 SW_Push, SW17 SW_Push, SW18 SW_Push, SW19 SW_Push, SW2 SW_Push, SW20 SW_Push, SW21 SW_Push, SW22 SW_Push, SW23 SW_Push, SW24 SW_Push, SW25 SW_Push, SW26 SW_Push, SW27 SW_Push, SW28 SW_Push, SW29 SW_Push, SW3 SW_Push, SW30 SW_Push, SW31 SW_Push, SW32 SW_Push, SW4 SW_Push, SW5 SW_Push, SW6 SW_Push, SW7 SW_Push, SW8 SW_Push, SW9 SW_Push, U1 LM358, U10 4051, U11 4051, U12 4051, U13 4051, U14 MicroSD_SPI_CD, U2 LM358, U3 Pico, U4 LM7805_TO220, U5 TL431LP, U6 4051, U7 PC817, U8 4051, U9 4051

Commit message: Code is added
Parts:
- R43, R71, R72, R73: value 1k -> 2k2
Connections:
- J8 pad G: unconnected-(J8-PadG) -> GND

Commit message: Fixes to midi circuit, added midi event handling
Parts:
- removed R67: 1k, Resistor_THT:R_Axial_DIN0207_L6.3mm_D2.5mm_P7.62mm_Horizontal
- R68: value 10k -> 2k2
- moved Q6 5.08 mm to (116.8, 59.5), turned to -90 degrees
- moved D3 3.05 mm to (99.8, 58.5)
- moved R62 3.05 mm to (99.8, 61.5)
Connections:
- U7 pad 3: Net-(R67-Pad2) -> Net-(Q6-Pad2)
Routing:
- net Net-(J11-Pad5): track 6.33 -> 26.8 mm
- net +3V3: track 255.9 -> 267.9 mm
- net Net-(Q6-Pad2): track 22.9 -> 30.0 mm
- net RX0: track 120.3 -> 126.7 mm
- net Net-(J11-Pad4): track 18.3 -> 12.5 mm
- net Net-(R67-Pad2): track 4.16 -> 0.00 mm
- net Net-(D3-Pad2): track 20.8 -> 23.8 mm
- net Net-(C40-Pad1): track 30.8 -> 32.8 mm

Commit message: Modified PCB, working sine synth
Parts:
- C12, C36, C8: value 2200 pF -> 22 nF
- C13, C37: value 470 pF -> 4700 pF
- C9: value 220 pF -> 2200 pF
- R10, R14, R15, R18, R19: value 10k -> 1k
- R11: value 100k -> 1k
- R13, R17: value 220k -> 22k
- R9: value 47k -> 4k7
- moved R68 15.8 mm to (111.5, 67.8)
- moved C16 13.2 mm to (149.9, 59.2), turned to -90 degrees
- moved C17 12.7 mm to (149.9, 67.6), turned to 90 degrees
- moved R17 7.67 mm to (144.8, 70.0)
- moved C11 6.50 mm to (141.4, 74.4)
- moved R13 3.73 mm to (138.3, 74.2)
- moved C28 3.26 mm to (142.3, 89.5)
- moved C10 3.14 mm to (149.4, 70.8), turned to -90 degrees
- moved U10 3.01 mm to (120.8, 97.6)
- moved C43 2.96 mm to (62.3, 90.1)
- moved U8 2.64 mm to (69.0, 97.2)
- moved C41 2.54 mm to (117.2, 91.6)
- moved R24 2.42 mm to (64.2, 87.0)
- moved D1 2.27 mm to (125.6, 68.5)
- moved C44 1.79 mm to (91.3, 90.9)
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Routing:
- net GND: track 34.6 -> 506.3 mm, vias 0 -> 46
- net Net-(Q6-Pad2): track 30.0 -> 15.4 mm
- net Net-(C36-Pad2): track 58.4 -> 67.1 mm
- net +3V3: track 267.9 -> 260.8 mm
- net Net-(C11-Pad1): track 9.89 -> 3.27 mm
- net FROMDAC2: track 51.5 -> 46.8 mm
- net BUTTON1: track 230.2 -> 234.2 mm
- net FROMDAC1: track 46.0 -> 49.4 mm
- net Net-(RV8-Pad2): track 11.7 -> 8.56 mm
- net CTRLB: track 263.1 -> 266.2 mm
- net Net-(RV13-Pad2): track 24.4 -> 21.4 mm
- net Net-(RV7-Pad2): track 24.0 -> 21.2 mm
- net Net-(RV14-Pad2): track 34.8 -> 32.0 mm
- net Net-(RV15-Pad2): track 24.1 -> 26.8 mm
- net Net-(C9-Pad1): track 14.4 -> 17.0 mm
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Other:
- board text added: "TrebleSynth by Daniel Marks VERSION 2 CC-BY-SA 4.0"
- board text removed: "TrebleSynth by Daniel Marks VERSION 1 CC-BY-SA 4.0"
