File: TrebleSynth/TrebleSynth.kicad_pcb (KiCad board)
At the start: 2 copper layers, 236 x 128 mm, 219 parts, among them J1 INPUT, J10 DIN-5_180degree, J11 DIN-5_180degree, J2 INPUT, J3 OUTPUT, J5 Barrel_Jack_Switch, J8 INPUT, J9 INPUT, Q1 2N3904, Q2 2N3904, Q3 2N3904, Q4 2N3904, Q5 2N3904, Q6 2N3904, SW1 SW_Push, SW10 SW_Push, SW11 SW_Push, SW12 SW_Push, SW13 SW_Push, SW14 SW_Push, SW15 SW_Push, SW16 SW_Push, SW17 SW_Push, SW18 SW_Push, SW19 SW_Push, SW2 SW_Push, SW20 SW_Push, SW21 SW_Push, SW22 SW_Push, SW23 SW_Push, SW24 SW_Push, SW25 SW_Push, SW26 SW_Push, SW27 SW_Push, SW28 SW_Push, SW29 SW_Push, SW3 SW_Push, SW30 SW_Push, SW31 SW_Push, SW32 SW_Push, SW4 SW_Push, SW5 SW_Push, SW6 SW_Push, SW7 SW_Push, SW8 SW_Push, SW9 SW_Push, U1 LM358, U10 4051, U11 4051, U12 4051, U13 4051, U14 MicroSD_SPI_CD, U2 LM358, U3 Pico, U4 LM7805_TO220, U5 TL431LP, U6 4051, U7 PC817, U8 4051, U9 4051

Commit message: Added pullup to MOSI
Parts:
- added R67: 10k, Resistor_THT:R_Axial_DIN0207_L6.3mm_D2.5mm_P7.62mm_Horizontal, F.Cu at (154.9, 49.4)
- R69: value 150R -> 220R
- moved C47 2.42 mm to (161.8, 41.7)
- moved C32 1.43 mm to (157.1, 46.0)
Routing:
- net MISO: track 44.8 -> 60.4 mm
- net +3V3: track 260.8 -> 266.3 mm
- net TX0: track 66.5 -> 70.6 mm
- net RX0: track 126.9 -> 130.1 mm
- net +5V: track 704.3 -> 707.3 mm
- net MOSI: track 47.3 -> 48.2 mm
- net SCK: track 44.5 -> 45.1 mm

Commit message: Added extra 3V3 capacitor
Parts:
- added C48: 100 nF, Capacitor_THT:C_Disc_D5.0mm_W2.5mm_P5.00mm, F.Cu at (138.6, 73.7)
- moved R13 3.67 mm to (139.2, 77.8)
- moved R14 2.49 mm to (87.7, 79.6)
- moved C13 2.47 mm to (72.7, 79.6)
- moved R35 0.71 mm to (193.5, 75.2)
- moved R33 0.65 mm to (193.5, 72.1)
- moved R34 0.64 mm to (191.2, 75.1)
- moved R30 0.64 mm to (191.2, 68.8)
- moved R28 0.62 mm to (191.2, 65.7)
- moved R32 0.59 mm to (191.2, 72.0)
- moved C21 0.59 mm to (100.6, 78.7)
- moved R31 0.54 mm to (193.5, 68.9)
- moved R29 0.48 mm to (193.6, 65.7)
Routing:
- net Net-(C12-Pad2): track 55.6 -> 59.5 mm
- net Net-(C13-Pad1): track 47.1 -> 49.6 mm
- net +3V3: track 266.3 -> 263.9 mm
- net SCL: track 76.1 -> 74.0 mm
- net Net-(C11-Pad1): track 3.27 -> 4.65 mm
- net Net-(C36-Pad2): track 67.1 -> 68.4 mm
- net Net-(R35-Pad2): track 16.4 -> 17.1 mm
- net FROMDAC1: track 49.4 -> 48.7 mm
- net RX0: track 130.1 -> 129.4 mm
- net Net-(R33-Pad2): track 17.0 -> 17.7 mm
- net Net-(C21-Pad1): track 26.2 -> 26.8 mm
- net Net-(R29-Pad2): track 17.2 -> 17.8 mm
- net Net-(R31-Pad2): track 16.9 -> 17.5 mm

Commit message: Added some more ground traces
Parts:
- moved R36 1.57 mm to (190.9, 46.3)
- moved R49 0.86 mm to (191.3, 52.8)
- moved R37 0.76 mm to (193.6, 47.8)
- moved R58 0.73 mm to (201.2, 44.7)
- moved R63 0.37 mm to (144.8, 58.0)
Routing:
- net GND: track 506.3 -> 689.5 mm, vias 46 -> 75
- net +3V3: track 263.9 -> 255.7 mm, vias 2 -> 3
- net SCL: track 74.0 -> 70.5 mm
- net SDA: track 62.5 -> 64.2 mm
- net SCK: track 45.1 -> 46.5 mm
- net MISO: track 60.4 -> 61.8 mm
- net SPICS: track 51.3 -> 52.6 mm
- net MOSI: track 48.2 -> 49.4 mm
- net Net-(Brd1-Pad2): track 52.2 -> 52.7 mm
