File: TrebleSynth/TrebleSynth.kicad_pcb (KiCad board)
At the start: 2 copper layers, 236 x 128 mm, 221 parts, among them J1 INPUT, J10 DIN-5_180degree, J11 DIN-5_180degree, J2 INPUT, J3 OUTPUT, J5 Barrel_Jack_Switch, J8 INPUT, J9 INPUT, Q1 2N3904, Q2 2N3904, Q3 2N3904, Q4 2N3904, Q5 2N3904, Q6 2N3904, SW1 SW_Push, SW10 SW_Push, SW11 SW_Push, SW12 SW_Push, SW13 SW_Push, SW14 SW_Push, SW15 SW_Push, SW16 SW_Push, SW17 SW_Push, SW18 SW_Push, SW19 SW_Push, SW2 SW_Push, SW20 SW_Push, SW21 SW_Push, SW22 SW_Push, SW23 SW_Push, SW24 SW_Push, SW25 SW_Push, SW26 SW_Push, SW27 SW_Push, SW28 SW_Push, SW29 SW_Push, SW3 SW_Push, SW30 SW_Push, SW31 SW_Push, SW32 SW_Push, SW4 SW_Push, SW5 SW_Push, SW6 SW_Push, SW7 SW_Push, SW8 SW_Push, SW9 SW_Push, U1 LM358, U10 4051, U11 4051, U12 4051, U13 4051, U14 MicroSD_SPI_CD, U2 LM358, U3 Pico, U4 LM7805_TO220, U5 TL431LP, U6 4051, U7 PC817, U8 4051, U9 4051

Commit message: Added some more ground traces
Parts:
- moved C48 5.09 mm to (133.5, 74.3)
Routing:
- net +3V3: track 255.7 -> 254.3 mm
- net Net-(C36-Pad2): track 68.7 -> 69.6 mm

Commit message: Tweaked the MIDI serial circuit again
Parts:
- added R74: 100R, Resistor_THT:R_Axial_DIN0207_L6.3mm_D2.5mm_P7.62mm_Horizontal, F.Cu at (138.9, 74.5)
- C48: value 100 nF -> 100 uF; footprint Capacitor_THT:C_Disc_D5.0mm_W2.5mm_P5.00mm -> Capacitor_THT:CP_Radial_D5.0mm_P2.50mm
- moved C19 28.9 mm to (149.6, 49.1)
- moved C48 5.29 mm to (130.6, 69.9), turned to 0 degrees
- moved C10 1.82 mm to (149.8, 72.6)
- moved C16 1.66 mm to (150.4, 60.8)
- moved C24 1.60 mm to (152.1, 58.1)
- moved C11 1.44 mm to (142.9, 74.4)
- moved C17 1.40 mm to (149.8, 69.0)
- moved R17 0.65 mm to (145.5, 70.1)
- moved R57 0.37 mm to (146.4, 55.5)
- moved R61 0.19 mm to (134.3, 65.7)
Connections:
- C48 pad 1: GND -> Net-(R69-Pad2)
- C48 pad 2: +3V3 -> GND
- R69 pad 2: +3V3 -> Net-(R69-Pad2)
- U7 pad 4: +3V3 -> Net-(R69-Pad2)
Routing:
- net +3V3: track 254.3 -> 217.8 mm
- net Net-(R69-Pad2): track 0.00 -> 31.9 mm
- net +5V: track 707.2 -> 702.9 mm
- net Net-(C36-Pad2): track 69.6 -> 68.2 mm
- net Net-(C17-Pad1): track 6.07 -> 4.78 mm
- net Net-(C10-Pad2): track 5.93 -> 4.70 mm
- net FROMDAC2: track 46.5 -> 45.3 mm
- net FROMDAC1: track 48.7 -> 48.1 mm
- net Net-(C11-Pad1): track 4.65 -> 5.22 mm
- net Net-(Brd1-Pad2): track 52.7 -> 53.3 mm
- net GND: track 689.5 -> 688.9 mm, vias 75 -> 72
- net RX0: track 129.6 -> 129.0 mm

Commit message: Changed schematic
Parts:
- R13, R17: value 22k -> 1k
- R27: value 1k -> 100R
