File: TrebleSynth/TrebleSynth.kicad_sch (KiCad schematic)
At the start: 126 parts, among them J1 INPUT, J10 DIN-5_180degree, J11 DIN-5_180degree, J2 INPUT, J3 OUTPUT, J5 Barrel_Jack_Switch, Q4 2N3904, Q5 2N3904, Q6 2N3904, U1 LM358, U2 LM358, U3 Pico, U4 LM7805_TO220, U5 TL431LP, U7 PC817

Commit message: Added SD card
Parts:
- added C47: 100 nF, Capacitor_THT:C_Disc_D5.0mm_W2.5mm_P5.00mm, symbol Device:C_Small
- added U14: MicroSD_SPI_CD, TrebleSynth:GCT-MEM2055-00-190-01-A, symbol microsd_spi_cd:MicroSD_SPI_CD
Connections:
- net +3V3: now also C47.1, U14.4 (VDD)
- net GND: now also C47.2, U14.6 (GND)
- net SCK: now reaches U3.4 (GPIO2)
- net SCK: now also U14.5 (SCLK)
- net MOSI: now reaches U3.5 (GPIO3)
- net MOSI: now also U14.3 (DI)
- net MISO: now reaches U3.6 (GPIO4)
- net MISO: now also U14.7 (DO)
- net SPICS: now reaches U3.7 (GPIO5)
- net SPICS: now also U14.2 (~{CS})

Commit message: Before moving around controls
Parts:
- added H10, H11, H12, H9: MountingHole, MountingHole:MountingHole_3.2mm_M3, symbol Mechanical:MountingHole
Other:
- moved on the sheet: H8
Changed lines of the file:
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@@
     (stroke (width 0) (type default) (color 0 0 0 0))
   )
-  (wire (pts (xy 88.265 163.83) (xy 88.265 167.005))
-    (stroke (width 0) (type default) (color 0 0 0 0))
-  )
   (wire (pts (xy 223.52 56.515) (xy 233.045 56.515))
     (stroke (width 0) (type default) (color 0 0 0 0))
@@
     )
   )
+  (symbol (lib_id "Mechanical:MountingHole") (at 114.935 153.035 0) (unit 1)
+    (in_bom yes) (on_board yes) (fields_autoplaced)
+    (property "Reference" "H11" (id 0) (at 117.475 151.7649 0)
+      (effects (font (size 1.27 1.27)) (justify left))
+    )
+    (property "Value" "MountingHole" (id 1) (at 117.475 154.3049 0)
+      (effects (font (size 1.27 1.27)) (justify left))
+    )
+    (property "Footprint" "MountingHole:MountingHole_3.2mm_M3" (id 2) (at 114.935 153.035 0)
+      (effects (font (size 1.27 1.27)) hide)
+    )
+    (property "Datasheet" "~" (id 3) (at 114.935 153.035 0)
+      (effects (font (size 1.27 1.27)) hide)
+    )
+  )
   (symbol (lib_id "Device:R") (at 159.385 31.115 270) (unit 1)
     (in_bom yes) (on_board yes)
@@
     (pin "2")
   )
+  (symbol (lib_id "Mechanical:MountingHole") (at 95.885 153.035 0) (unit 1)
+    (in_bom yes) (on_board yes) (fields_autoplaced)
+    (property "Reference" "H9" (id 0) (at 98.425 151.7649 0)
+      (effects (font (size 1.27 1.27)) (justify left))
+    )
+    (property "Value" "MountingHole" (id 1) (at 98.425 154.3049 0)
+      (effects (font (size 1.27 1.27)) (justify left))
+    )
+    (property "Footprint" "MountingHole:MountingHole_3.2mm_M3" (id 2) (at 95.885 153.035 0)
+      (effects (font (size 1.27 1.27)) hide)
+    )
+    (property "Datasheet" "~" (id 3) (at 95.885 153.035 0)
+      (effects (font (size 1.27 1.27)) hide)
+    )
+  )
   (symbol (lib_id "Device:C_Polarized_Small") (at 90.805 123.825 90) (unit 1)
     (in_bom yes) (on_board yes) (fields_autoplaced)
@@
     (pin "2")
   )
-  (symbol (lib_id "power:+5V") (at 88.265 163.83 0) (unit 1)
+  (symbol (lib_id "power:+5V") (at 88.265 167.005 0) (unit 1)
     (in_bom yes) (on_board yes) (fields_autoplaced)
-    (property "Reference" "#PWR0111" (id 0) (at 88.265 167.64 0)
+    (property "Reference" "#PWR0111" (id 0) (at 88.265 170.815 0)
       (effects (font (size 1.27 1.27)) hide)
     )
-    (property "Value" "+5V" (id 1) (at 88.265 158.75 0))
-    (property "Footprint" "" (id 2) (at 88.265 163.83 0)
+    (property "Value" "+5V" (id 1) (at 88.265 161.925 0))
+    (property "Footprint" "" (id 2) (at 88.265 167.005 0)
       (effects (font (size 1.27 1.27)) hide)
     )
-    (property "Datasheet" "" (id 3) (at 88.265 163.83 0)
+    (property "Datasheet" "" (id 3) (at 88.265 167.005 0)
       (effects (font (size 1.27 1.27)) hide)
     )
     (pin "1")
   )
+  (symbol (lib_id "Mechanical:MountingHole") (at 95.885 159.385 0) (unit 1)
+    (in_bom yes) (on_board yes) (fields_autoplaced)
+    (property "Reference" "H10" (id 0) (at 98.425 158.1149 0)
+      (effects (font (size 1.27 1.27)) (justify left))
+    )
+    (property "Value" "MountingHole" (id 1) (at 98.425 160.6549 0)
+      (effects (font (size 1.27 1.27)) (justify left))
+    )
+    (property "Footprint" "MountingHole:MountingHole_3.2mm_M3" (id 2) (at 95.885 159.385 0)
+      (effects (font (size 1.27 1.27)) hide)
+    )
+    (property "Datasheet" "~" (id 3) (at 95.885 159.385 0)
+      (effects (font (size 1.27 1.27)) hide)
+    )
+  )
   (symbol (lib_id "Device:R") (at 74.93 50.165 270) (unit 1)
     (in_bom yes) (on_board yes)
@@
     (pin "2")
   )
-  (symbol (lib_id "Mechanical:MountingHole") (at 95.885 153.035 0) (unit 1)
+  (symbol (lib_id "Mechanical:MountingHole") (at 76.835 158.75 0) (unit 1)
     (in_bom yes) (on_board yes) (fields_autoplaced)
-    (property "Reference" "H8" (id 0) (at 98.425 151.7649 0)
+    (property "Reference" "H8" (id 0) (at 79.375 157.4799 0)
       (effects (font (size 1.27 1.27)) (justify left))
     )
-    (property "Value" "MountingHole" (id 1) (at 98.425 154.3049 0)
+    (property "Value" "MountingHole" (id 1) (at 79.375 160.0199 0)
       (effects (font (size 1.27 1.27)) (justify left))
     )
-    (property "Footprint" "MountingHole:MountingHole_3.2mm_M3" (id 2) (at 95.885 153.035 0)
+    (property "Footprint" "MountingHole:MountingHole_3.2mm_M3" (id 2) (at 76.835 158.75 0)
       (effects (font (size 1.27 1.27)) hide)
     )
-    (property "Datasheet" "~" (id 3) (at 95.885 153.035 0)
+    (property "Datasheet" "~" (id 3) (at 76.835 158.75 0)
       (effects (font (size 1.27 1.27)) hide)
     )
@@
     (pin "1")
   )
+  (symbol (lib_id "Mechanical:MountingHole") (at 114.935 159.385 0) (unit 1)
+    (in_bom yes) (on_board yes) (fields_autoplaced)
+    (property "Reference" "H12" (id 0) (at 117.475 158.1149 0)
+      (effects (font (size 1.27 1.27)) (justify left))
+    )
+    (property "Value" "MountingHole" (id 1) (at 117.475 160.6549 0)
+      (effects (font (size 1.27 1.27)) (justify left))
+    )
+    (property "Footprint" "MountingHole:MountingHole_3.2mm_M3" (id 2) (at 114.935 159.385 0)
+      (effects (font (size 1.27 1.27)) hide)
+    )
+    (property "Datasheet" "~" (id 3) (at 114.935 159.385 0)
+      (effects (font (size 1.27 1.27)) hide)
+    )
+  )
   (symbol (lib_id "Device:R") (at 170.18 31.115 90) (unit 1)
     (in_bom yes) (on_board yes)
@@
       (reference "H8") (unit 1) (value "MountingHole") (footprint "MountingHole:MountingHole_3.2mm_M3")
     )
+    (path "/64759d19-a147-49e9-a4da-f2d91645074a"
+      (reference "H9") (unit 1) (value "MountingHole") (footprint "MountingHole:MountingHole_3.2mm_M3")
+    )
+    (path "/8d9a8770-00ad-4771-b49f-dc6cda59e35f"
+      (reference "H10") (unit 1) (value "MountingHole") (footprint "MountingHole:MountingHole_3.2mm_M3")
+    )
+    (path "/001a75ac-1454-4c6d-90f9-fbe6874d5531"
+      (reference "H11") (unit 1) (value "MountingHole") (footprint "MountingHole:MountingHole_3.2mm_M3")
+    )
+    (path "/be0fd112-576d-42ad-8276-a5c84089edca"
+      (reference "H12") (unit 1) (value "MountingHole") (footprint "MountingHole:MountingHole_3.2mm_M3")
+    )
     (path "/af9e4a9a-836c-4e54-ad12-e6879e1054f7"

Commit message: Fixes to midi circuit, added midi event handling
Parts:
- removed R67: 1k, Resistor_THT:R_Axial_DIN0207_L6.3mm_D2.5mm_P7.62mm_Horizontal, symbol Device:R
- R68: value 10k -> 2k2
Connections:
- net at Q6.2 (B), R68.2: now also U7.3
Changed lines of the file:
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@@
     (stroke (width 0) (type default) (color 0 0 0 0))
   )
-  (wire (pts (xy 209.55 98.425) (xy 209.55 99.06))
-    (stroke (width 0) (type default) (color 0 0 0 0))
-  )
   (wire (pts (xy 273.05 37.465) (xy 273.685 37.465))
     (stroke (width 0) (type default) (color 0 0 0 0))
@@
     (stroke (width 0) (type default) (color 0 0 0 0))
   )
-  (wire (pts (xy 228.6 116.205) (xy 228.6 117.475))
+  (wire (pts (xy 228.6 108.585) (xy 228.6 117.475))
     (stroke (width 0) (type default) (color 0 0 0 0))
   )
@@
     (pin "G")
   )
-  (symbol (lib_id "Device:R") (at 228.6 112.395 180) (unit 1)
-    (in_bom yes) (on_board yes)
-    (property "Reference" "R67" (id 0) (at 231.013 110.998 90)
-      (effects (font (size 1.27 1.27)) (justify left))
-    )
-    (property "Value" "1k" (id 1) (at 228.6 111.125 90)
-      (effects (font (size 1.27 1.27)) (justify left))
-    )
-    (property "Footprint" "Resistor_THT:R_Axial_DIN0207_L6.3mm_D2.5mm_P7.62mm_Horizontal" (id 2) (at 230.378 112.395 90)
-      (effects (font (size 1.27 1.27)) hide)
-    )
-    (property "Datasheet" "~" (id 3) (at 228.6 112.395 0)
-      (effects (font (size 1.27 1.27)) hide)
-    )
-    (pin "1")
-    (pin "2")
-  )
   (symbol (lib_id "Device:C_Small") (at 241.935 53.34 0) (unit 1)
     (in_bom yes) (on_board yes)
@@
       (effects (font (size 1.27 1.27)) (justify left))
     )
-    (property "Value" "10k" (id 1) (at 228.6 120.015 90)
+    (property "Value" "2k2" (id 1) (at 228.6 120.015 90)
       (effects (font (size 1.27 1.27)) (justify left))
     )
@@
       (reference "R66") (unit 1) (value "220R") (footprint "Resistor_THT:R_Axial_DIN0207_L6.3mm_D2.5mm_P7.62mm_Horizontal")
     )
-    (path "/151856d4-577e-4f0e-b641-ad358fd86c64"
-      (reference "R67") (unit 1) (value "1k") (footprint "Resistor_THT:R_Axial_DIN0207_L6.3mm_D2.5mm_P7.62mm_Horizontal")
-    )
     (path "/e00de198-ef3a-420b-ab26-e3557c5dcced"
-      (reference "R68") (unit 1) (value "10k") (footprint "Resistor_THT:R_Axial_DIN0207_L6.3mm_D2.5mm_P7.62mm_Horizontal")
+      (reference "R68") (unit 1) (value "2k2") (footprint "Resistor_THT:R_Axial_DIN0207_L6.3mm_D2.5mm_P7.62mm_Horizontal")
     )
     (path "/5af5c4be-8a48-495b-97c9-d05f389cff3d"

Commit message: Modified PCB, working sine synth
Parts:
- C12, C36, C8: value 2200 pF -> 22 nF
- C13, C37: value 470 pF -> 4700 pF
- C9: value 220 pF -> 2200 pF
- R10, R14, R15, R18, R19: value 10k -> 1k
- R11: value 100k -> 1k
- R13, R17: value 220k -> 22k
- R9: value 47k -> 4k7
Changed lines of the file:
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@@
       (effects (font (size 1.27 1.27)) (justify left))
     )
-    (property "Value" "100k" (id 1) (at 121.539 50.292 90)
+    (property "Value" "1k" (id 1) (at 122.555 50.165 90)
       (effects (font (size 1.27 1.27)) (justify left))
     )
@@
       (effects (font (size 1.27 1.27)) (justify left))
     )
-    (property "Value" "10k" (id 1) (at 55.88 126.365 90)
+    (property "Value" "1k" (id 1) (at 55.88 126.365 90)
       (effects (font (size 1.27 1.27)) (justify left))
     )
@@
     (in_bom yes) (on_board yes)
     (property "Reference" "C9" (id 0) (at 123.19 40.64 90))
-    (property "Value" "220 pF" (id 1) (at 123.19 46.99 90))
+    (property "Value" "2200 pF" (id 1) (at 123.19 46.99 90))
     (property "Footprint" "Capacitor_THT:C_Disc_D5.0mm_W2.5mm_P5.00mm" (id 2) (at 123.19 43.815 0)
       (effects (font (size 1.27 1.27)) hide)
@@
       (effects (font (size 1.27 1.27)) (justify left))
     )
-    (property "Value" "10k" (id 1) (at 110.49 38.1 90)
+    (property "Value" "1k" (id 1) (at 110.49 38.1 90)
       (effects (font (size 1.27 1.27)) (justify left))
     )
@@
       (effects (font (size 1.27 1.27)) (justify left))
     )
-    (property "Value" "220k" (id 1) (at 44.45 84.455 90)
+    (property "Value" "22k" (id 1) (at 43.815 84.455 90)
       (effects (font (size 1.27 1.27)) (justify left))
     )
@@
   )
   (symbol (lib_id "Device:C_Small") (at 47.625 121.285 0) (unit 1)
-    (in_bom yes) (on_board yes) (fields_autoplaced)
+    (in_bom yes) (on_board yes)
     (property "Reference" "C36" (id 0) (at 50.8 120.0212 0)
       (effects (font (size 1.27 1.27)) (justify left))
     )
-    (property "Value" "2200 pF" (id 1) (at 50.8 122.5612 0)
+    (property "Value" "22 nF" (id 1) (at 50.165 121.92 0)
       (effects (font (size 1.27 1.27)) (justify left))
     )
@@
     (in_bom yes) (on_board yes)
     (property "Reference" "C37" (id 0) (at 69.215 132.715 90))
-    (property "Value" "470 pF" (id 1) (at 69.215 139.065 90))
+    (property "Value" "4700 pF" (id 1) (at 69.215 139.065 90))
     (property "Footprint" "Capacitor_THT:C_Disc_D5.0mm_W2.5mm_P5.00mm" (id 2) (at 69.215 135.89 0)
       (effects (font (size 1.27 1.27)) hide)
@@
   (symbol (lib_id "Device:C_Small") (at 102.87 33.655 0) (unit 1)
     (in_bom yes) (on_board yes) (fields_autoplaced)
-    (property "Reference" "C8" (id 0) (at 105.283 32.3912 0)
+    (property "Reference" "C8" (id 0) (at 105.41 32.3912 0)
       (effects (font (size 1.27 1.27)) (justify left))
     )
-    (property "Value" "2200 pF" (id 1) (at 105.283 34.9312 0)
+    (property "Value" "22 nF" (id 1) (at 105.41 34.9312 0)
       (effects (font (size 1.27 1.27)) (justify left))
     )
@@
       (effects (font (size 1.27 1.27)) (justify left))
     )
-    (property "Value" "10k" (id 1) (at 55.245 84.455 90)
+    (property "Value" "1k" (id 1) (at 55.245 84.455 90)
       (effects (font (size 1.27 1.27)) (justify left))
     )
@@
   )
   (symbol (lib_id "Device:C_Small") (at 46.99 79.375 0) (unit 1)
-    (in_bom yes) (on_board yes) (fields_autoplaced)
-    (property "Reference" "C12" (id 0) (at 50.165 78.1112 0)
+    (in_bom yes) (on_board yes)
+    (property "Reference" "C12" (id 0) (at 49.53 78.1112 0)
       (effects (font (size 1.27 1.27)) (justify left))
     )
-    (property "Value" "2200 pF" (id 1) (at 50.165 80.6512 0)
+    (property "Value" "22 nF" (id 1) (at 49.53 80.01 0)
       (effects (font (size 1.27 1.27)) (justify left))
     )
@@
       (effects (font (size 1.27 1.27)) (justify left))
     )
-    (property "Value" "47k" (id 1) (at 100.33 38.1 90)
+    (property "Value" "4k7" (id 1) (at 100.33 38.1 90)
       (effects (font (size 1.27 1.27)) (justify left))
     )
@@
       (effects (font (size 1.27 1.27)) (justify left))
     )
-    (property "Value" "10k" (id 1) (at 69.85 100.965 90)
+    (property "Value" "1k" (id 1) (at 69.85 100.965 90)
       (effects (font (size 1.27 1.27)) (justify left))
     )
@@
       (effects (font (size 1.27 1.27)) (justify left))
     )
-    (property "Value" "10k" (id 1) (at 70.485 142.875 90)
+    (property "Value" "1k" (id 1) (at 70.485 142.875 90)
       (effects (font (size 1.27 1.27)) (justify left))
     )
@@
       (effects (font (size 1.27 1.27)) (justify left))
     )
-    (property "Value" "220k" (id 1) (at 45.085 126.365 90)
+    (property "Value" "22k" (id 1) (at 44.45 126.365 90)
       (effects (font (size 1.27 1.27)) (justify left))
     )
@@
     (in_bom yes) (on_board yes)
     (property "Reference" "C13" (id 0) (at 68.58 90.805 90))
-    (property "Value" "470 pF" (id 1) (at 68.58 97.155 90))
+    (property "Value" "4700 pF" (id 1) (at 68.58 97.155 90))
     (property "Footprint" "Capacitor_THT:C_Disc_D5.0mm_W2.5mm_P5.00mm" (id 2) (at 68.58 93.98 0)
       (effects (font (size 1.27 1.27)) hide)
@@
     )
     (path "/7c8415b8-7547-4704-bf1c-41e45abebbf6"
-      (reference "C8") (unit 1) (value "2200 pF") (footprint "Capacitor_THT:C_Disc_D5.0mm_W2.5mm_P5.00mm")
+      (reference "C8") (unit 1) (value "22 nF") (footprint "Capacitor_THT:C_Disc_D5.0mm_W2.5mm_P5.00mm")
     )
     (path "/1d2e8b1f-46b0-47a7-a4b5-d2612d2633f0"
-      (reference "C9") (unit 1) (value "220 pF") (footprint "Capacitor_THT:C_Disc_D5.0mm_W2.5mm_P5.00mm")
+      (reference "C9") (unit 1) (value "2200 pF") (footprint "Capacitor_THT:C_Disc_D5.0mm_W2.5mm_P5.00mm")
     )
     (path "/2e8ce526-6fc8-4bf6-8e88-01110c5fb478"
@@
     )
     (path "/944a30cb-00bd-425f-b8d2-7613a7bc143d"
-      (reference "C12") (unit 1) (value "2200 pF") (footprint "Capacitor_THT:C_Disc_D5.0mm_W2.5mm_P5.00mm")
+      (reference "C12") (unit 1) (value "22 nF") (footprint "Capacitor_THT:C_Disc_D5.0mm_W2.5mm_P5.00mm")
     )
     (path "/f9e582af-f7a7-46da-b838-4d87800ad119"
-      (reference "C13") (unit 1) (value "470 pF") (footprint "Capacitor_THT:C_Disc_D5.0mm_W2.5mm_P5.00mm")
+      (reference "C13") (unit 1) (value "4700 pF") (footprint "Capacitor_THT:C_Disc_D5.0mm_W2.5mm_P5.00mm")
     )
     (path "/7b62232e-dc1b-424a-bd96-df5531b112a2"
@@
     )
     (path "/5c4e5dc7-449c-427d-a54c-031606e1c69c"
-      (reference "C36") (unit 1) (value "2200 pF") (footprint "Capacitor_THT:C_Disc_D5.0mm_W2.5mm_P5.00mm")
+      (reference "C36") (unit 1) (value "22 nF") (footprint "Capacitor_THT:C_Disc_D5.0mm_W2.5mm_P5.00mm")
     )
     (path "/63417ad5-d0e8-4c57-aa08-e78b33106b04"
-      (reference "C37") (unit 1) (value "470 pF") (footprint "Capacitor_THT:C_Disc_D5.0mm_W2.5mm_P5.00mm")
+      (reference "C37") (unit 1) (value "4700 pF") (footprint "Capacitor_THT:C_Disc_D5.0mm_W2.5mm_P5.00mm")
     )
     (path "/6726b8b1-03cc-40f6-8f36-06dff53c78e7"
@@
     )
     (path "/d4beb8d8-4bc5-47e7-9fb4-402e9c122e28"
-      (reference "R9") (unit 1) (value "47k") (footprint "Resistor_THT:R_Axial_DIN0207_L6.3mm_D2.5mm_P7.62mm_Horizontal")
+      (reference "R9") (unit 1) (value "4k7") (footprint "Resistor_THT:R_Axial_DIN0207_L6.3mm_D2.5mm_P7.62mm_Horizontal")
     )
     (path "/34f11cdf-c071-4cc5-a787-48df288af0ba"
-      (reference "R10") (unit 1) (value "10k") (footprint "Resistor_THT:R_Axial_DIN0207_L6.3mm_D2.5mm_P7.62mm_Horizontal")
+      (reference "R10") (unit 1) (value "1k") (footprint "Resistor_THT:R_Axial_DIN0207_L6.3mm_D2.5mm_P7.62mm_Horizontal")
     )
     (path "/136aa926-be0e-4d47-8f5a-3e755b401e00"
-      (reference "R11") (unit 1) (value "100k") (footprint "Resistor_THT:R_Axial_DIN0207_L6.3mm_D2.5mm_P7.62mm_Horizontal")
+      (reference "R11") (unit 1) (value "1k") (footprint "Resistor_THT:R_Axial_DIN0207_L6.3mm_D2.5mm_P7.62mm_Horizontal")
     )
     (path "/9949ef93-2cf9-4b67-a871-53f2bebedd68"
@@
     )
     (path "/497e8e16-db24-4b63-b1a9-654c978540b6"
-      (reference "R13") (unit 1) (value "220k") (footprint "Resistor_THT:R_Axial_DIN0207_L6.3mm_D2.5mm_P7.62mm_Horizontal")
+      (reference "R13") (unit 1) (value "22k") (footprint "Resistor_THT:R_Axial_DIN0207_L6.3mm_D2.5mm_P7.62mm_Horizontal")
     )
     (path "/8311fdd2-488f-44b2-97f8-bec3fa3e522a"
-      (reference "R14") (unit 1) (value "10k") (footprint "Resistor_THT:R_Axial_DIN0207_L6.3mm_D2.5mm_P7.62mm_Horizontal")
+      (reference "R14") (unit 1) (value "1k") (footprint "Resistor_THT:R_Axial_DIN0207_L6.3mm_D2.5mm_P7.62mm_Horizontal")
     )
     (path "/dee588ca-cd6f-49bd-8482-b92f631940ad"
-      (reference "R15") (unit 1) (value "10k") (footprint "Resistor_THT:R_Axial_DIN0207_L6.3mm_D2.5mm_P7.62mm_Horizontal")
+      (reference "R15") (unit 1) (value "1k") (footprint "Resistor_THT:R_Axial_DIN0207_L6.3mm_D2.5mm_P7.62mm_Horizontal")
     )
     (path "/f985247c-ef50-4b7d-a7ba-9d9ed0bb0d70"
@@
     )
     (path "/ecfd8248-9c56-4fdf-99f7-d731692babfd"
-      (reference "R17") (unit 1) (value "220k") (footprint "Resistor_THT:R_Axial_DIN0207_L6.3mm_D2.5mm_P7.62mm_Horizontal")
+      (reference "R17") (unit 1) (value "22k") (footprint "Resistor_THT:R_Axial_DIN0207_L6.3mm_D2.5mm_P7.62mm_Horizontal")
     )
     (path "/174a1aa8-a61d-404d-bf38-4a43145f8086"
-      (reference "R18") (unit 1) (value "10k") (footprint "Resistor_THT:R_Axial_DIN0207_L6.3mm_D2.5mm_P7.62mm_Horizontal")
+      (reference "R18") (unit 1) (value "1k") (footprint "Resistor_THT:R_Axial_DIN0207_L6.3mm_D2.5mm_P7.62mm_Horizontal")
     )
     (path "/e02e27fd-948a-4355-bbc5-10290f6ac8af"
-      (reference "R19") (unit 1) (value "10k") (footprint "Resistor_THT:R_Axial_DIN0207_L6.3mm_D2.5mm_P7.62mm_Horizontal")
+      (reference "R19") (unit 1) (value "1k") (footprint "Resistor_THT:R_Axial_DIN0207_L6.3mm_D2.5mm_P7.62mm_Horizontal")
     )
     (path "/20df9d49-7795-4085-9a0d-1460a2c1c7cf"

Commit message: Before removing interrupt poll
Parts:
- R69: value 150R -> 220R
Changed lines of the file:
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@@
       (effects (font (size 1.27 1.27)) (justify left))
     )
-    (property "Value" "150R" (id 1) (at 236.22 104.14 90)
+    (property "Value" "220R" (id 1) (at 236.22 104.14 90)
       (effects (font (size 1.27 1.27)) (justify left))
     )
@@
     )
     (path "/5af5c4be-8a48-495b-97c9-d05f389cff3d"
-      (reference "R69") (unit 1) (value "150R") (footprint "Resistor_THT:R_Axial_DIN0207_L6.3mm_D2.5mm_P7.62mm_Horizontal")
+      (reference "R69") (unit 1) (value "220R") (footprint "Resistor_THT:R_Axial_DIN0207_L6.3mm_D2.5mm_P7.62mm_Horizontal")
     )
     (path "/7c0a3443-6e78-4c33-b3f2-c6e5539da31b/1f458ea9-c23d-4695-850e-e5d48e78d85e"
