File: TrebleSynth/TrebleSynth.kicad_sch (KiCad schematic)
At the start: 131 parts, among them J1 INPUT, J10 DIN-5_180degree, J11 DIN-5_180degree, J2 INPUT, J3 OUTPUT, J5 Barrel_Jack_Switch, Q4 2N3904, Q5 2N3904, Q6 2N3904, U1 LM358, U14 MicroSD_SPI_CD, U2 LM358, U3 Pico, U4 LM7805_TO220, U5 TL431LP, U7 PC817

Commit message: Added pullup to MOSI
Parts:
- added R67: 10k, Resistor_THT:R_Axial_DIN0207_L6.3mm_D2.5mm_P7.62mm_Horizontal, symbol Device:R
Connections:
- net +3V3: now also R67.1
- net MISO: now also R67.2
Other:
- moved on the sheet: U14
Changed lines of the file:
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@@
   (junction (at 46.99 75.565) (diameter 0) (color 0 0 0 0)
   )
+  (junction (at 257.81 94.615) (diameter 0) (color 0 0 0 0)
+  )
   (junction (at 236.22 125.095) (diameter 0) (color 0 0 0 0)
   )
@@
     (stroke (width 0) (type default) (color 0 0 0 0))
   )
+  (wire (pts (xy 257.81 94.615) (xy 261.62 94.615))
+    (stroke (width 0) (type default) (color 0 0 0 0))
+  )
   (wire (pts (xy 62.23 167.005) (xy 65.405 167.005))
     (stroke (width 0) (type default) (color 0 0 0 0))
@@
     (stroke (width 0) (type default) (color 0 0 0 0))
   )
-  (wire (pts (xy 241.3 86.995) (xy 255.27 86.995))
+  (wire (pts (xy 257.81 71.12) (xy 257.81 73.025))
+    (stroke (width 0) (type default) (color 0 0 0 0))
+  )
+  (wire (pts (xy 241.3 86.995) (xy 261.62 86.995))
     (stroke (width 0) (type default) (color 0 0 0 0))
   )
@@
     (stroke (width 0) (type default) (color 0 0 0 0))
   )
-  (wire (pts (xy 250.825 89.535) (xy 255.27 89.535))
+  (wire (pts (xy 250.825 89.535) (xy 261.62 89.535))
     (stroke (width 0) (type default) (color 0 0 0 0))
   )
@@
     (stroke (width 0) (type default) (color 0 0 0 0))
   )
+  (wire (pts (xy 257.81 80.645) (xy 257.81 94.615))
+    (stroke (width 0) (type default) (color 0 0 0 0))
+  )
   (wire (pts (xy 175.895 48.895) (xy 187.96 48.895))
     (stroke (width 0) (type default) (color 0 0 0 0))
@@
     (stroke (width 0) (type default) (color 0 0 0 0))
   )
-  (wire (pts (xy 252.73 92.075) (xy 255.27 92.075))
+  (wire (pts (xy 252.73 92.075) (xy 261.62 92.075))
     (stroke (width 0) (type default) (color 0 0 0 0))
   )
@@
     (stroke (width 0) (type default) (color 0 0 0 0))
   )
-  (wire (pts (xy 252.095 81.915) (xy 255.27 81.915))
+  (wire (pts (xy 252.095 81.915) (xy 261.62 81.915))
     (stroke (width 0) (type default) (color 0 0 0 0))
   )
@@
     (stroke (width 0) (type default) (color 0 0 0 0))
   )
-  (wire (pts (xy 251.46 84.455) (xy 255.27 84.455))
+  (wire (pts (xy 251.46 84.455) (xy 261.62 84.455))
     (stroke (width 0) (type default) (color 0 0 0 0))
   )
-  (wire (pts (xy 251.46 94.615) (xy 255.27 94.615))
+  (wire (pts (xy 251.46 94.615) (xy 257.81 94.615))
     (stroke (width 0) (type default) (color 0 0 0 0))
   )
@@
     (pin "2")
   )
-  (symbol (lib_id "microsd_spi_cd:MicroSD_SPI_CD") (at 264.16 89.535 0) (mirror y) (unit 1)
+  (symbol (lib_id "microsd_spi_cd:MicroSD_SPI_CD") (at 270.51 89.535 0) (mirror y) (unit 1)
     (in_bom yes) (on_board yes) (fields_autoplaced)
-    (property "Reference" "U14" (id 0) (at 271.78 88.265 0)
+    (property "Reference" "U14" (id 0) (at 278.13 88.265 0)
       (effects (font (size 1.524 1.524)) (justify right))
     )
-    (property "Value" "MicroSD_SPI_CD" (id 1) (at 271.78 92.075 0)
+    (property "Value" "MicroSD_SPI_CD" (id 1) (at 278.13 92.075 0)
       (effects (font (size 1.524 1.524)) (justify right))
     )
-    (property "Footprint" "TrebleSynth:GCT-MEM2055-00-190-01-A" (id 2) (at 264.16 77.47 0)
+    (property "Footprint" "TrebleSynth:GCT-MEM2055-00-190-01-A" (id 2) (at 270.51 77.47 0)
       (effects (font (size 1.524 1.524)) hide)
     )
-    (property "Datasheet" "" (id 3) (at 267.97 89.535 0)
+    (property "Datasheet" "" (id 3) (at 274.32 89.535 0)
       (effects (font (size 1.524 1.524)))
     )
@@
     (pin "1")
   )
+  (symbol (lib_id "power:+3V3") (at 257.81 71.12 0) (unit 1)
+    (in_bom yes) (on_board yes) (fields_autoplaced)
+    (property "Reference" "#PWR0180" (id 0) (at 257.81 74.93 0)
+      (effects (font (size 1.27 1.27)) hide)
+    )
+    (property "Value" "+3V3" (id 1) (at 257.81 66.04 0))
+    (property "Footprint" "" (id 2) (at 257.81 71.12 0)
+      (effects (font (size 1.27 1.27)) hide)
+    )
+    (property "Datasheet" "" (id 3) (at 257.81 71.12 0)
+      (effects (font (size 1.27 1.27)) hide)
+    )
+    (pin "1")
+  )
   (symbol (lib_id "power:+5V") (at 197.485 133.35 0) (unit 1)
     (in_bom yes) (on_board yes)
@@
     (pin "1")
   )
+  (symbol (lib_id "Device:R") (at 257.81 76.835 0) (unit 1)
+    (in_bom yes) (on_board yes)
+    (property "Reference" "R67" (id 0) (at 255.905 78.74 90)
+      (effects (font (size 1.27 1.27)) (justify left))
+    )
+    (property "Value" "10k" (id 1) (at 257.81 78.105 90)
+      (effects (font (size 1.27 1.27)) (justify left))
+    )
+    (property "Footprint" "Resistor_THT:R_Axial_DIN0207_L6.3mm_D2.5mm_P7.62mm_Horizontal" (id 2) (at 256.032 76.835 90)
+      (effects (font (size 1.27 1.27)) hide)
+    )
+    (property "Datasheet" "~" (id 3) (at 257.81 76.835 0)
+      (effects (font (size 1.27 1.27)) hide)
+    )
+    (pin "1")
+    (pin "2")
+  )
   (symbol (lib_id "Mechanical:MountingHole") (at 95.885 159.385 0) (unit 1)
     (in_bom yes) (on_board yes) (fields_autoplaced)
@@
       (reference "#PWR0179") (unit 1) (value "GND") (footprint "")
     )
+    (path "/70a17b1b-0631-4990-9538-580f761e1ecf"
+      (reference "#PWR0180") (unit 1) (value "+3V3") (footprint "")
+    )
     (path "/7c0a3443-6e78-4c33-b3f2-c6e5539da31b/d4632855-44e2-4d51-9d69-5a3b7dc301aa"
       (reference "#PWR0181") (unit 1) (value "GND") (footprint "")
@@
       (reference "R66") (unit 1) (value "220R") (footprint "Resistor_THT:R_Axial_DIN0207_L6.3mm_D2.5mm_P7.62mm_Horizontal")
     )
+    (path "/8a74cad7-05ad-476d-a88b-1574ab05a258"
+      (reference "R67") (unit 1) (value "10k") (footprint "Resistor_THT:R_Axial_DIN0207_L6.3mm_D2.5mm_P7.62mm_Horizontal")
+    )
     (path "/e00de198-ef3a-420b-ab26-e3557c5dcced"

Commit message: Added extra 3V3 capacitor
Parts:
- added C48: 100 nF, Capacitor_THT:C_Disc_D5.0mm_W2.5mm_P5.00mm, symbol Device:C_Small
Connections:
- net +3V3: now also C48.2
- net GND: now also C48.1
Changed lines of the file:
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@@
   (junction (at 165.1 62.23) (diameter 0) (color 0 0 0 0)
   )
+  (junction (at 236.22 102.87) (diameter 0) (color 0 0 0 0)
+  )
   (junction (at 149.86 149.225) (diameter 0) (color 0 0 0 0)
   )
@@
     (stroke (width 0) (type default) (color 0 0 0 0))
   )
+  (wire (pts (xy 248.92 125.095) (xy 236.22 125.095))
+    (stroke (width 0) (type default) (color 0 0 0 0))
+  )
   (wire (pts (xy 135.89 141.605) (xy 135.89 139.7))
     (stroke (width 0) (type default) (color 0 0 0 0))
@@
     (stroke (width 0) (type default) (color 0 0 0 0))
   )
+  (wire (pts (xy 248.92 114.3) (xy 248.92 125.095))
+    (stroke (width 0) (type default) (color 0 0 0 0))
+  )
   (wire (pts (xy 131.445 131.445) (xy 131.445 141.605))
     (stroke (width 0) (type default) (color 0 0 0 0))
@@
     (stroke (width 0) (type default) (color 0 0 0 0))
   )
+  (wire (pts (xy 248.92 102.87) (xy 248.92 109.22))
+    (stroke (width 0) (type default) (color 0 0 0 0))
+  )
   (wire (pts (xy 163.195 53.975) (xy 164.465 53.975))
     (stroke (width 0) (type default) (color 0 0 0 0))
@@
     (stroke (width 0) (type default) (color 0 0 0 0))
   )
+  (wire (pts (xy 236.22 102.87) (xy 248.92 102.87))
+    (stroke (width 0) (type default) (color 0 0 0 0))
+  )
   (wire (pts (xy 204.47 114.935) (xy 204.47 113.665))
     (stroke (width 0) (type default) (color 0 0 0 0))
@@
     (pin "2")
   )
+  (symbol (lib_id "Device:C_Small") (at 248.92 111.76 180) (unit 1)
+    (in_bom yes) (on_board yes)
+    (property "Reference" "C48" (id 0) (at 253.365 113.665 0)
+      (effects (font (size 1.27 1.27)) (justify left))
+    )
+    (property "Value" "100 nF" (id 1) (at 256.54 109.855 0)
+      (effects (font (size 1.27 1.27)) (justify left))
+    )
+    (property "Footprint" "Capacitor_THT:C_Disc_D5.0mm_W2.5mm_P5.00mm" (id 2) (at 248.92 111.76 0)
+      (effects (font (size 1.27 1.27)) hide)
+    )
+    (property "Datasheet" "~" (id 3) (at 248.92 111.76 0)
+      (effects (font (size 1.27 1.27)) hide)
+    )
+    (pin "1")
+    (pin "2")
+  )
   (symbol (lib_id "power:GND") (at 215.9 153.035 0) (unit 1)
     (in_bom yes) (on_board yes) (fields_autoplaced)
@@
       (reference "C47") (unit 1) (value "100 nF") (footprint "Capacitor_THT:C_Disc_D5.0mm_W2.5mm_P5.00mm")
     )
+    (path "/20eec51e-6e74-4173-a9eb-203c9177b7d2"
+      (reference "C48") (unit 1) (value "100 nF") (footprint "Capacitor_THT:C_Disc_D5.0mm_W2.5mm_P5.00mm")
+    )
     (path "/c47f2778-675e-4a19-8402-9385e9308b9c"
