File: TrebleSynth/TrebleSynth.kicad_sch (KiCad schematic)
At the start: 133 parts, among them J1 INPUT, J10 DIN-5_180degree, J11 DIN-5_180degree, J2 INPUT, J3 OUTPUT, J5 Barrel_Jack_Switch, Q4 2N3904, Q5 2N3904, Q6 2N3904, U1 LM358, U14 MicroSD_SPI_CD, U2 LM358, U3 Pico, U4 LM7805_TO220, U5 TL431LP, U7 PC817

Commit message: Tweaked the MIDI serial circuit again
Parts:
- removed C48: 100 nF, Capacitor_THT:C_Disc_D5.0mm_W2.5mm_P5.00mm, symbol Device:C_Small
- added C48: 100 uF, Capacitor_THT:CP_Radial_D5.0mm_P2.50mm, symbol Device:C_Polarized_Small
- added R74: 100R, Resistor_THT:R_Axial_DIN0207_L6.3mm_D2.5mm_P7.62mm_Horizontal, symbol Device:R
Connections:
- net +3V3: now also R74.1; no longer R69.2, U7.4
- net GND: now also C48.2
- new net: C48.1, R69.2, R74.2, U7.4
Changed lines of the file:
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@@
     (pin "2")
   )
-  (symbol (lib_id "Device:C_Small") (at 248.92 111.76 180) (unit 1)
-    (in_bom yes) (on_board yes)
-    (property "Reference" "C48" (id 0) (at 253.365 113.665 0)
-      (effects (font (size 1.27 1.27)) (justify left))
-    )
-    (property "Value" "100 nF" (id 1) (at 256.54 109.855 0)
-      (effects (font (size 1.27 1.27)) (justify left))
-    )
-    (property "Footprint" "Capacitor_THT:C_Disc_D5.0mm_W2.5mm_P5.00mm" (id 2) (at 248.92 111.76 0)
-      (effects (font (size 1.27 1.27)) hide)
-    )
-    (property "Datasheet" "~" (id 3) (at 248.92 111.76 0)
-      (effects (font (size 1.27 1.27)) hide)
-    )
-    (pin "1")
-    (pin "2")
-  )
   (symbol (lib_id "power:GND") (at 215.9 153.035 0) (unit 1)
     (in_bom yes) (on_board yes) (fields_autoplaced)
@@
     (pin "4")
   )
+  (symbol (lib_id "Device:C_Polarized_Small") (at 248.92 111.76 0) (unit 1)
+    (in_bom yes) (on_board yes) (fields_autoplaced)
+    (property "Reference" "C48" (id 0) (at 251.46 109.9438 0)
+      (effects (font (size 1.27 1.27)) (justify left))
+    )
+    (property "Value" "100 uF" (id 1) (at 251.46 112.4838 0)
+      (effects (font (size 1.27 1.27)) (justify left))
+    )
+    (property "Footprint" "Capacitor_THT:CP_Radial_D5.0mm_P2.50mm" (id 2) (at 248.92 111.76 0)
+      (effects (font (size 1.27 1.27)) hide)
+    )
+    (property "Datasheet" "~" (id 3) (at 248.92 111.76 0)
+      (effects (font (size 1.27 1.27)) hide)
+    )
+    (pin "1")
+    (pin "2")
+  )
   (symbol (lib_id "power:+3V3") (at 241.3 78.74 0) (unit 1)
     (in_bom yes) (on_board yes) (fields_autoplaced)
@@
     (pin "2")
   )
-  (symbol (lib_id "power:+3V3") (at 228.6 99.695 0) (unit 1)
+  (symbol (lib_id "power:+3V3") (at 228.6 92.075 0) (unit 1)
     (in_bom yes) (on_board yes) (fields_autoplaced)
-    (property "Reference" "#PWR0164" (id 0) (at 228.6 103.505 0)
+    (property "Reference" "#PWR0164" (id 0) (at 228.6 95.885 0)
       (effects (font (size 1.27 1.27)) hide)
     )
-    (property "Value" "+3V3" (id 1) (at 228.6 94.615 0))
-    (property "Footprint" "" (id 2) (at 228.6 99.695 0)
+    (property "Value" "+3V3" (id 1) (at 228.6 86.995 0))
+    (property "Footprint" "" (id 2) (at 228.6 92.075 0)
       (effects (font (size 1.27 1.27)) hide)
     )
-    (property "Datasheet" "" (id 3) (at 228.6 99.695 0)
+    (property "Datasheet" "" (id 3) (at 228.6 92.075 0)
       (effects (font (size 1.27 1.27)) hide)
     )
@@
     (pin "2")
   )
+  (symbol (lib_id "Device:R") (at 228.6 95.885 0) (unit 1)
+    (in_bom yes) (on_board yes)
+    (property "Reference" "R74" (id 0) (at 226.187 97.282 90)
+      (effects (font (size 1.27 1.27)) (justify left))
+    )
+    (property "Value" "100R" (id 1) (at 228.6 98.425 90)
+      (effects (font (size 1.27 1.27)) (justify left))
+    )
+    (property "Footprint" "Resistor_THT:R_Axial_DIN0207_L6.3mm_D2.5mm_P7.62mm_Horizontal" (id 2) (at 226.822 95.885 90)
+      (effects (font (size 1.27 1.27)) hide)
+    )
+    (property "Datasheet" "~" (id 3) (at 228.6 95.885 0)
+      (effects (font (size 1.27 1.27)) hide)
+    )
+    (pin "1")
+    (pin "2")
+  )
   (symbol (lib_id "Device:C_Small") (at 25.4 177.165 0) (unit 1)
     (in_bom yes) (on_board yes) (fields_autoplaced)
@@
       (reference "C47") (unit 1) (value "100 nF") (footprint "Capacitor_THT:C_Disc_D5.0mm_W2.5mm_P5.00mm")
     )
-    (path "/20eec51e-6e74-4173-a9eb-203c9177b7d2"
-      (reference "C48") (unit 1) (value "100 nF") (footprint "Capacitor_THT:C_Disc_D5.0mm_W2.5mm_P5.00mm")
+    (path "/389a2061-ad0d-44cc-98bf-076f67892f1c"
+      (reference "C48") (unit 1) (value "100 uF") (footprint "Capacitor_THT:CP_Radial_D5.0mm_P2.50mm")
     )
     (path "/c47f2778-675e-4a19-8402-9385e9308b9c"
@@
       (reference "R73") (unit 1) (value "2k2") (footprint "Resistor_THT:R_Axial_DIN0207_L6.3mm_D2.5mm_P7.62mm_Horizontal")
     )
+    (path "/fc2f6805-0ec3-4e3a-a457-c5c3c61a1c71"
+      (reference "R74") (unit 1) (value "100R") (footprint "Resistor_THT:R_Axial_DIN0207_L6.3mm_D2.5mm_P7.62mm_Horizontal")
+    )
     (path "/1fba26fe-d2f2-4acc-9daa-6e3d6c311e42"

Commit message: Changed schematic
Parts:
- R13, R17: value 22k -> 1k
- R27: value 1k -> 100R
