File: TrebleSynth/TrebleSynthControls.kicad_sch (KiCad schematic)
At the start: 88 parts, among them J8 INPUT, J9 INPUT, Q1 2N3904, Q2 2N3904, Q3 2N3904, SW1 SW_Push, SW10 SW_Push, SW11 SW_Push, SW12 SW_Push, SW13 SW_Push, SW14 SW_Push, SW15 SW_Push, SW16 SW_Push, SW17 SW_Push, SW18 SW_Push, SW19 SW_Push, SW2 SW_Push, SW20 SW_Push, SW21 SW_Push, SW22 SW_Push, SW23 SW_Push, SW24 SW_Push, SW25 SW_Push, SW26 SW_Push, SW27 SW_Push, SW28 SW_Push, SW29 SW_Push, SW3 SW_Push, SW30 SW_Push, SW31 SW_Push, SW32 SW_Push, SW4 SW_Push, SW5 SW_Push, SW6 SW_Push, SW7 SW_Push, SW8 SW_Push, SW9 SW_Push, U10 4051, U11 4051, U12 4051, U13 4051, U6 4051, U8 4051, U9 4051

Commit message: Code is added
Parts:
- R43, R71, R72, R73: value 1k -> 2k2
Connections:
- net GND: now also J8.G
Changed lines of the file:
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@@
     (pin "2")
+  )
+  (symbol (lib_id "power:GND") (at 183.515 52.705 0) (unit 1)
+    (in_bom yes) (on_board yes) (fields_autoplaced)
+    (property "Reference" "#PWR0153" (id 0) (at 183.515 59.055 0)
+      (effects (font (size 1.27 1.27)) hide)
+    )
+    (property "Value" "GND" (id 1) (at 183.515 57.15 0))
+    (property "Footprint" "" (id 2) (at 183.515 52.705 0)
+      (effects (font (size 1.27 1.27)) hide)
+    )
+    (property "Datasheet" "" (id 3) (at 183.515 52.705 0)
+      (effects (font (size 1.27 1.27)) hide)
+    )
+    (pin "1")
   )
   (symbol (lib_id "power:+5V") (at 52.07 111.125 0) (unit 1)
@@
       (effects (font (size 1.27 1.27)) (justify left))
     )
-    (property "Value" "1k" (id 1) (at 64.77 116.205 90)
+    (property "Value" "2k2" (id 1) (at 64.77 116.205 90)
       (effects (font (size 1.27 1.27)) (justify left))
     )
@@
       (effects (font (size 1.27 1.27)) (justify left))
     )
-    (property "Value" "1k" (id 1) (at 124.46 118.11 90)
+    (property "Value" "2k2" (id 1) (at 124.46 118.11 90)
       (effects (font (size 1.27 1.27)) (justify left))
     )
@@
       (effects (font (size 1.27 1.27)) (justify left))
     )
-    (property "Value" "1k" (id 1) (at 242.57 118.11 90)
+    (property "Value" "2k2" (id 1) (at 242.57 118.11 90)
       (effects (font (size 1.27 1.27)) (justify left))
     )
@@
       (effects (font (size 1.27 1.27)) (justify left))
     )
-    (property "Value" "1k" (id 1) (at 184.15 118.11 90)
-      (effects (font (size 1.27 1.27)) (justify left))
-    )
+    (property "Value" "2k2" (id 1) (at 184.15 118.11 90)
+      (effects (font (size 1.27 1.27)) (justify left))
+    )
